File: KiCad/icescreamer.kicad_pcb (KiCad board)
At the start: 2 copper layers, 49.5 x 57.1 mm, 47 parts, among them CON1 PWR_IN, J1 JACK, J2 JACK, P1 BAT_T, Q1 NPN, Q2 NPN, SW1 3PDT, U1 TL072

Commit message: Updated WIP pcb
Parts:
- moved R15 115.2 mm to (52.1, 120.7)
- moved R16 104.2 mm to (64.8, 124.5)
- moved R19 99.8 mm to (53.3, 128.3)
- moved R17 91.7 mm to (76.2, 127.0)
- moved R12 89.8 mm to (40.6, 129.5)
- moved R1 83.6 mm to (40.6, 114.3)
- moved R2 83.1 mm to (40.6, 121.9)
- moved R18 78.2 mm to (86.4, 127.0)
- moved J1 78.1 mm to (40.6, 49.5), turned to 0 degrees
- moved C1 73.4 mm to (21.6, 104.1)
- moved C11 71.9 mm to (34.3, 108.0)
- moved J2 42.2 mm to (43.2, 90.2)
- moved C9 41.1 mm to (81.4, 73.7)
- moved D4 40.2 mm to (97.8, 53.3)
- moved R10 39.1 mm to (78.7, 83.8)
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Routing:
- net GND: track 157.0 -> 18.0 mm, vias 2 -> 0
- net FX in: track 124.7 -> 0.00 mm, vias 3 -> 0
- net Net-(C4-Pad2): track 119.2 -> 46.0 mm
- net -5V: track 129.4 -> 60.3 mm, vias 2 -> 0
- net FX out: track 64.8 -> 0.00 mm
- net Net-(Q2-Pad1): track 62.0 -> 4.56 mm
- net +5V: track 147.7 -> 90.9 mm
- net Net-(J2-PadT): track 54.3 -> 0.00 mm, vias 1 -> 0
- net Net-(C3-Pad1): track 84.4 -> 33.5 mm, vias 1 -> 0
- net Net-(R19-Pad2): track 50.4 -> 0.00 mm, vias 1 -> 0
- net Net-(R11-Pad1): track 45.8 -> 0.00 mm, vias 1 -> 0
- net Net-(CON1-Pad1): track 44.7 -> 0.00 mm
- net Net-(D3-Pad1): track 43.1 -> 0.00 mm, vias 1 -> 0
- net Net-(J1-PadT): track 42.9 -> 0.00 mm
- net Net-(C6-Pad2): track 0.00 -> 40.3 mm
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